Commit message: fix: robot_model import ok!

File: core/robot_model/test_robot/urdf/test_robot.urdf (robot description, URDF)
Before this commit: robot test_robot, 12 links, 11 joints
Links:
- link J1_link: mass 0.847544109052372 -> 0.847544109052371
- link J2_link: mass 1.0271 -> 1.51834737973212
- link J3_link: mass 0.521461387664207 -> 0.705419071317585
- link J4_link: mass 0.155182108030077 -> 0.269784889847788
- link J5_link: mass 0.163676857530181 -> 0.284892561638528
- link left_after_link: mass 0.19255 -> 0.192554360111192
- link left_befor_link: mass 0.24322 -> 0.243221956120782
- link right_after_link: mass 0.243221922457797 -> 0.243221956118719
- link right_before_link: mass 0.192554332103213 -> 0.192554360118823
- link robot_base_link: mass 2.876 -> 3.6973552164338
Joints:
- joint J1_joint: origin xyz=0.1893 0.07 0.0029078 rpy=1.5708 1.5708 0 -> xyz=0.189301311254835 0.07 0.00290782987848454 rpy=-1.5707963267949 1.5707963267949 0
- joint J2_joint: origin xyz=0.016827 -0.079897 0.102 rpy=-1.5708 0 0.20757 -> xyz=0.0815435988166945 -0.00416701236161837 0.102 rpy=-1.5707963267949 0 1.51973909018581
- joint J3_joint: origin xyz=-0.1971 -0.26467 0.0289 rpy=0 0 0 -> xyz=-0.297380428115131 -0.143055517104597 0.0288999999999909 rpy=0 0 0
- joint J4_joint: origin xyz=-0.052059 0.11529 0.055 rpy=1.5708 0.2271 0.42414 -> xyz=-0.0520591601532436 0.1152913433183 0.0550000000000078 rpy=1.57079632679501 1.52425622041413 0.424137505817387
- joint J5_joint: origin xyz=0.015079 -0.039735 -0.06 rpy=-1.5708 -0.43982 0.3627 -> xyz=0.0423315447474402 0.00378025386648639 -0.0600000000000362 rpy=1.5707963267949 -0.231927791500107 -1.48173147181141
- joint J6_joint: origin xyz=-0.15612 -0.045077 -0.0155 rpy=0 0 0 -> xyz=0.150256395086882 -0.0618810612020733 -0.0155000000000037 rpy=0 0 0
- joint J7_joint: origin xyz=-0.0024297 0.060952 0.0516 rpy=1.5708 0.331 0.039842 -> xyz=-0.0394368251984132 -0.0465374775666559 0.0515999999999899 rpy=-1.57079632679491 1.50090735517209 -0.702994782778823
- joint left_after_join: origin xyz=-0.14707 -0.038473 -0.2485 rpy=0 0 -3.1416 -> xyz=-0.147074515694654 -0.0384729858248051 -0.248499619316574 rpy=0 0 -3.14159265358979
- joint left_befor_joint: origin xyz=0.23 -0.038473 -0.2485 rpy=0 0 -3.1416 -> xyz=0.229997401922067 -0.0384729858248118 -0.248499619316559 rpy=0 0 -3.14159265358979
- joint right_after_joint: origin xyz=-0.14707 -0.038473 0.2607 rpy=0 1.5708 0 -> xyz=-0.14707451569465 -0.0384729858248003 0.260700380683427 rpy=0 1.5707963267949 0
- joint right_before_joint: origin xyz=0.23 -0.038473 0.2607 rpy=3.1416 0 3.1416 -> xyz=0.229997401922066 -0.0384729858248047 0.260700380683427 rpy=3.14159265358979 0 3.14159265358979

Commit message: fix: import a new model and run demo ok

File: core/robot_model/test_robot/urdf/test_robot.urdf (robot description, URDF)
Before this commit: robot test_robot, 12 links, 11 joints
Joints:
- removed joint left_after_join
- removed joint left_befor_joint
- added joint left_after_joint: type continuous, parent robot_base_link, child left_after_link, origin xyz=-0.147074515694654 -0.0384729858248051 -0.248499619316574 rpy=0 0 -3.14159265358979, axis 0 0 -1
- added joint left_before_joint: type continuous, parent robot_base_link, child left_befor_link, origin xyz=0.229997401922067 -0.0384729858248118 -0.248499619316559 rpy=0 0 -3.14159265358979, axis 0 0 -1

Commit message: fix: 彻底解决了测试模型的问题，除了关于麦轮的配置

File: core/robot_model/test_robot/urdf/test_robot.urdf (robot description, URDF)
Before this commit: robot test_robot, 12 links, 11 joints
Links:
- link J1_link: mass 0.847544109052371 -> 1.23425990593155
- link J2_link: mass 1.51834737973212 -> 1.10586856399633
- link J3_link: mass 0.705419071317585 -> 0.538855476414292
- link J4_link: mass 0.269784889847788 -> 0.172878482049537
- link J5_link: mass 0.284892561638528 -> 0.18220557422278
- link left_after_link: mass 0.192554360111192 -> 0.192554371338558
- link left_befor_link: mass 0.243221956120782 -> 0.243221967341035
- link right_after_link: mass 0.243221956118719 -> 0.243221967338972
- link right_before_link: mass 0.192554360118823 -> 0.192554371346189
- link robot_base_link: mass 3.6973552164338 -> 3.72431445026937
Joints:
- joint J1_joint: origin xyz=0.189301311254835 0.07 0.00290782987848454 rpy=-1.5707963267949 1.5707963267949 0 -> xyz=0.147839868141125 0.00319255080494721 0.108472985824806 rpy=0 0 1.5707963267949
- joint J6_joint: origin xyz=0.150256395086882 -0.0618810612020733 -0.0155000000000037 rpy=0 0 0 -> xyz=0.15026 -0.061881 -0.0155 rpy=0 0 0
- joint J7_joint: origin xyz=-0.0394368251984132 -0.0465374775666559 0.0515999999999899 rpy=-1.57079632679491 1.50090735517209 -0.702994782778823 -> xyz=-0.039437 -0.046537 0.0516 rpy=-1.5708 1.5009 -0.70299
- joint left_after_joint: origin xyz=-0.147074515694654 -0.0384729858248051 -0.248499619316574 rpy=0 0 -3.14159265358979 -> xyz=-0.188535958808364 0.254600000000006 0 rpy=-1.5707963267949 0 -3.14159265358979
- joint left_before_joint: origin xyz=0.229997401922067 -0.0384729858248118 -0.248499619316559 rpy=0 0 -3.14159265358979 -> xyz=0.188535958808357 0.254599999999991 0 rpy=-1.5707963267949 0 3.14159265358978
- joint right_after_joint: origin xyz=-0.14707451569465 -0.0384729858248003 0.260700380683427 rpy=0 1.5707963267949 0 -> xyz=-0.18853595880836 -0.254599999999995 0 rpy=1.5707963267949 0 1.5707963267949
- joint right_before_joint: origin xyz=0.229997401922066 -0.0384729858248047 0.260700380683427 rpy=3.14159265358979 0 3.14159265358979 -> xyz=0.188535958808356 -0.254599999999996 0 rpy=1.5707963267949 0 3.14159265358978

File: core/robot_model/test_robot_moveit/config/test_robot.ros2_control.xacro (robot description, xacro)
@@ -8,91 +8,123 @@
                 <plugin>mock_components/GenericSystem</plugin>
             </hardware>
+            <joint name="robot_base_joint_virtual">
+                <command_interface name="position"/>
+                <command_interface name="velocity"/>
+                <command_interface name="effort"/>
+                <state_interface name="position">
+                  <param name="initial_value">${initial_positions['robot_base_joint_virtual']}</param>
+                </state_interface>
+                <state_interface name="velocity"/>
+                <state_interface name="effort"/>
+            </joint>
             <joint name="J1_joint">
                 <command_interface name="position"/>
+                <command_interface name="velocity"/>
+                <command_interface name="effort"/>
                 <state_interface name="position">
                   <param name="initial_value">${initial_positions['J1_joint']}</param>
                 </state_interface>
                 <state_interface name="velocity"/>
+                <state_interface name="effort"/>
             </joint>
             <joint name="J2_joint">
                 <command_interface name="position"/>
+                <command_interface name="velocity"/>
+                <command_interface name="effort"/>
                 <state_interface name="position">
                   <param name="initial_value">${initial_positions['J2_joint']}</param>
                 </state_interface>
                 <state_interface name="velocity"/>
+                <state_interface name="effort"/>
             </joint>
             <joint name="J3_joint">
                 <command_interface name="position"/>
+                <command_interface name="velocity"/>
+                <command_interface name="effort"/>
                 <state_interface name="position">
                   <param name="initial_value">${initial_positions['J3_joint']}</param>
                 </state_interface>
                 <state_interface name="velocity"/>
+                <state_interface name="effort"/>
             </joint>
             <joint name="J4_joint">
                 <command_interface name="position"/>
+                <command_interface name="velocity"/>
+                <command_interface name="effort"/>
                 <state_interface name="position">
                   <param name="initial_value">${initial_positions['J4_joint']}</param>
                 </state_interface>
                 <state_interface name="velocity"/>
+                <state_interface name="effort"/>
             </joint>
             <joint name="J5_joint">
                 <command_interface name="position"/>
+                <command_interface name="velocity"/>
+                <command_interface name="effort"/>
                 <state_interface name="position">
                   <param name="initial_value">${initial_positions['J5_joint']}</param>
                 </state_interface>
                 <state_interface name="velocity"/>
+                <state_interface name="effort"/>
             </joint>
             <joint name="J6_joint">
                 <command_interface name="position"/>
+                <command_interface name="velocity"/>
+                <command_interface name="effort"/>
                 <state_interface name="position">
                   <param name="initial_value">${initial_positions['J6_joint']}</param>
                 </state_interface>
                 <state_interface name="velocity"/>
+                <state_interface name="effort"/>
             </joint>
             <joint name="J7_joint">
                 <command_interface name="position"/>
+                <command_interface name="velocity"/>
+                <command_interface name="effort"/>
                 <state_interface name="position">
                   <param name="initial_value">${initial_positions['J7_joint']}</param>
                 </state_interface>
                 <state_interface name="velocity"/>
-            </joint>
-            <joint name="robot_base_joint_virtual">
-                <command_interface name="position"/>
-                <state_interface name="position">
-                  <param name="initial_value">${initial_positions['robot_base_joint_virtual']}</param>
-                </state_interface>
-                <state_interface name="velocity"/>
+                <state_interface name="effort"/>
             </joint>
             <joint name="left_after_joint">
                 <command_interface name="position"/>
                 <command_interface name="velocity"/>
+                <command_interface name="effort"/>
                 <state_interface name="position">
                   <param name="initial_value">${initial_positions['left_after_joint']}</param>
                 </state_interface>
                 <state_interface name="velocity"/>
+                <state_interface name="effort"/>
             </joint>
             <joint name="left_before_joint">
                 <command_interface name="position"/>
                 <command_interface name="velocity"/>
+                <command_interface name="effort"/>
                 <state_interface name="position">
                   <param name="initial_value">${initial_positions['left_before_joint']}</param>
                 </state_interface>
                 <state_interface name="velocity"/>
+                <state_interface name="effort"/>
             </joint>
             <joint name="right_after_joint">
                 <command_interface name="position"/>
                 <command_interface name="velocity"/>
+                <command_interface name="effort"/>
                 <state_interface name="position">
                   <param name="initial_value">${initial_positions['right_after_joint']}</param>
                 </state_interface>
                 <state_interface name="velocity"/>
+                <state_interface name="effort"/>
             </joint>
             <joint name="right_before_joint">
                 <command_interface name="position"/>
                 <command_interface name="velocity"/>
+                <command_interface name="effort"/>
                 <state_interface name="position">
                   <param name="initial_value">${initial_positions['right_before_joint']}</param>
                 </state_interface>
                 <state_interface name="velocity"/>
+                <state_interface name="effort"/>
             </joint>
         </ros2_control>

Commit message: fix: 修复的机器人模型的问题，现在的问题是，麦轮控制器和moveit_controller 无法直接对接

File: core/robot_model/test_robot/urdf/test_robot.urdf (robot description, URDF)
Before this commit: robot test_robot, 12 links, 11 joints
Links:
- added link dummy
Joints:
- added joint dummy_joint: type fixed, parent dummy, child robot_base_link

File: core/robot_model/test_robot_moveit/config/test_robot.ros2_control.xacro (robot description, xacro)
@@ -8,123 +8,67 @@
                 <plugin>mock_components/GenericSystem</plugin>
             </hardware>
-            <joint name="robot_base_joint_virtual">
-                <command_interface name="position"/>
-                <command_interface name="velocity"/>
-                <command_interface name="effort"/>
-                <state_interface name="position">
-                  <param name="initial_value">${initial_positions['robot_base_joint_virtual']}</param>
-                </state_interface>
-                <state_interface name="velocity"/>
-                <state_interface name="effort"/>
-            </joint>
             <joint name="J1_joint">
                 <command_interface name="position"/>
                 <command_interface name="velocity"/>
-                <command_interface name="effort"/>
                 <state_interface name="position">
                   <param name="initial_value">${initial_positions['J1_joint']}</param>
                 </state_interface>
                 <state_interface name="velocity"/>
-                <state_interface name="effort"/>
             </joint>
             <joint name="J2_joint">
                 <command_interface name="position"/>
                 <command_interface name="velocity"/>
-                <command_interface name="effort"/>
                 <state_interface name="position">
                   <param name="initial_value">${initial_positions['J2_joint']}</param>
                 </state_interface>
                 <state_interface name="velocity"/>
-                <state_interface name="effort"/>
             </joint>
             <joint name="J3_joint">
                 <command_interface name="position"/>
                 <command_interface name="velocity"/>
-                <command_interface name="effort"/>
                 <state_interface name="position">
                   <param name="initial_value">${initial_positions['J3_joint']}</param>
                 </state_interface>
                 <state_interface name="velocity"/>
-                <state_interface name="effort"/>
             </joint>
             <joint name="J4_joint">
                 <command_interface name="position"/>
                 <command_interface name="velocity"/>
-                <command_interface name="effort"/>
                 <state_interface name="position">
                   <param name="initial_value">${initial_positions['J4_joint']}</param>
                 </state_interface>
                 <state_interface name="velocity"/>
-                <state_interface name="effort"/>
             </joint>
             <joint name="J5_joint">
                 <command_interface name="position"/>
                 <command_interface name="velocity"/>
-                <command_interface name="effort"/>
                 <state_interface name="position">
                   <param name="initial_value">${initial_positions['J5_joint']}</param>
                 </state_interface>
                 <state_interface name="velocity"/>
-                <state_interface name="effort"/>
             </joint>
             <joint name="J6_joint">
                 <command_interface name="position"/>
                 <command_interface name="velocity"/>
-                <command_interface name="effort"/>
                 <state_interface name="position">
                   <param name="initial_value">${initial_positions['J6_joint']}</param>
                 </state_interface>
                 <state_interface name="velocity"/>
-                <state_interface name="effort"/>
             </joint>
             <joint name="J7_joint">
                 <command_interface name="position"/>
                 <command_interface name="velocity"/>
-                <command_interface name="effort"/>
                 <state_interface name="position">
                   <param name="initial_value">${initial_positions['J7_joint']}</param>
                 </state_interface>
                 <state_interface name="velocity"/>
-                <state_interface name="effort"/>
             </joint>
-            <joint name="left_after_joint">
+            <joint name="dummy_virtual_joint">
                 <command_interface name="position"/>
                 <command_interface name="velocity"/>
-                <command_interface name="effort"/>
                 <state_interface name="position">
-                  <param name="initial_value">${initial_positions['left_after_joint']}</param>
+                  <param name="initial_value">${initial_positions['dummy_virtual_joint']}</param>
                 </state_interface>
                 <state_interface name="velocity"/>
-                <state_interface name="effort"/>
-            </joint>
-            <joint name="left_before_joint">
-                <command_interface name="position"/>
-                <command_interface name="velocity"/>
-                <command_interface name="effort"/>
-                <state_interface name="position">
-                  <param name="initial_value">${initial_positions['left_before_joint']}</param>
-                </state_interface>
-                <state_interface name="velocity"/>
-                <state_interface name="effort"/>
-            </joint>
-            <joint name="right_after_joint">
-                <command_interface name="position"/>
-                <command_interface name="velocity"/>
-                <command_interface name="effort"/>
-                <state_interface name="position">
-                  <param name="initial_value">${initial_positions['right_after_joint']}</param>
-                </state_interface>
-                <state_interface name="velocity"/>
-                <state_interface name="effort"/>
-            </joint>
-            <joint name="right_before_joint">
-                <command_interface name="position"/>
-                <command_interface name="velocity"/>
-                <command_interface name="effort"/>
-                <state_interface name="position">
-                  <param name="initial_value">${initial_positions['right_before_joint']}</param>
-                </state_interface>
-                <state_interface name="velocity"/>
-                <state_interface name="effort"/>
             </joint>
         </ros2_control>

Commit message: feature: 实现了启动文件的不同namespace配置

File: core/robot_model/test_robot/urdf/test_robot.urdf (robot description, URDF)
Before this commit: robot test_robot, 13 links, 12 joints
Links:
- link J1_link: geometry collision mesh filename=$(find test_robot)/meshes/J1_link.STL; visual mesh filename=$(find test_robot)/meshes/J1_link.STL
- link J2_link: geometry collision mesh filename=$(find test_robot)/meshes/J2_link.STL; visual mesh filename=$(find test_robot)/meshes/J2_link.STL
- link J3_link: geometry collision mesh filename=$(find test_robot)/meshes/J3_link.STL; visual mesh filename=$(find test_robot)/meshes/J3_link.STL
- link J4_link: geometry collision mesh filename=$(find test_robot)/meshes/J4_link.STL; visual mesh filename=$(find test_robot)/meshes/J4_link.STL
- link J5_link: geometry collision mesh filename=$(find test_robot)/meshes/J5_link.STL; visual mesh filename=$(find test_robot)/meshes/J5_link.STL
- link J6_link: geometry collision mesh filename=$(find test_robot)/meshes/J6_link.STL; visual mesh filename=$(find test_robot)/meshes/J6_link.STL
- link J7_link: geometry collision mesh filename=$(find test_robot)/meshes/J7_link.STL; visual mesh filename=$(find test_robot)/meshes/J7_link.STL
- link left_after_link: geometry collision mesh filename=$(find test_robot)/meshes/left_after_link.STL; visual mesh filename=$(find test_robot)/meshes/left_after_link.STL
- link left_befor_link: geometry collision mesh filename=$(find test_robot)/meshes/left_befor_link.STL; visual mesh filename=$(find test_robot)/meshes/left_befor_link.STL
- link right_after_link: geometry collision mesh filename=$(find test_robot)/meshes/right_after_link.STL; visual mesh filename=$(find test_robot)/meshes/right_after_link.STL
- link right_before_link: geometry collision mesh filename=$(find test_robot)/meshes/right_before_link.STL; visual mesh filename=$(find test_robot)/meshes/right_before_link.STL
- link robot_base_link: geometry collision mesh filename=$(find test_robot)/meshes/robot_base_link.STL; visual mesh filename=$(find test_robot)/meshes/robot_base_link.STL
Joints:
- joint dummy_joint: origin (none) -> xyz=0 0 0.1 rpy=0 0 0
- joint right_after_joint: axis -1 0 0 -> 1 0 0
- joint right_before_joint: axis 0 0 -1 -> 0 0 1
