Commit message: fix: 完善gazebo_test_model.py文件，使其可以直接使用原有urdf文件

File: core/robot_model/test_robot/urdf/test_robot.urdf (robot description, URDF)
Before this commit: robot test_robot, 13 links, 12 joints
Links:
- link J1_link: geometry collision mesh filename=package://test_robot/meshes/J1_link.STL; visual mesh filename=package://test_robot/meshes/J1_link.STL
- link J2_link: geometry collision mesh filename=package://test_robot/meshes/J2_link.STL; visual mesh filename=package://test_robot/meshes/J2_link.STL
- link J3_link: geometry collision mesh filename=package://test_robot/meshes/J3_link.STL; visual mesh filename=package://test_robot/meshes/J3_link.STL
- link J4_link: geometry collision mesh filename=package://test_robot/meshes/J4_link.STL; visual mesh filename=package://test_robot/meshes/J4_link.STL
- link J5_link: geometry collision mesh filename=package://test_robot/meshes/J5_link.STL; visual mesh filename=package://test_robot/meshes/J5_link.STL
- link J6_link: geometry collision mesh filename=package://test_robot/meshes/J6_link.STL; visual mesh filename=package://test_robot/meshes/J6_link.STL
- link J7_link: geometry collision mesh filename=package://test_robot/meshes/J7_link.STL; visual mesh filename=package://test_robot/meshes/J7_link.STL
- link left_after_link: geometry collision mesh filename=package://test_robot/meshes/left_after_link.STL; visual mesh filename=package://test_robot/meshes/left_after_link.STL
- link left_befor_link: geometry collision mesh filename=package://test_robot/meshes/left_befor_link.STL; visual mesh filename=package://test_robot/meshes/left_befor_link.STL
- link right_after_link: geometry collision mesh filename=package://test_robot/meshes/right_after_link.STL; visual mesh filename=package://test_robot/meshes/right_after_link.STL
- link right_before_link: geometry collision mesh filename=package://test_robot/meshes/right_before_link.STL; visual mesh filename=package://test_robot/meshes/right_before_link.STL
- link robot_base_link: geometry collision mesh filename=package://test_robot/meshes/robot_base_link.STL; visual mesh filename=package://test_robot/meshes/robot_base_link.STL

Commit message: fix: 成功实现了从moveit和gazebo的基础联合仿真

File: core/robot_model/test_robot/urdf/test_robot.urdf (robot description, URDF)
Before this commit: robot test_robot, 13 links, 12 joints
Links:
- link J1_link: geometry collision mesh filename=file://$(find test_robot)/meshes/J1_link.STL; visual mesh filename=file://$(find test_robot)/meshes/J1_link.STL
- link J2_link: geometry collision mesh filename=file://$(find test_robot)/meshes/J2_link.STL; visual mesh filename=file://$(find test_robot)/meshes/J2_link.STL
- link J3_link: geometry collision mesh filename=file://$(find test_robot)/meshes/J3_link.STL; visual mesh filename=file://$(find test_robot)/meshes/J3_link.STL
- link J4_link: geometry collision mesh filename=file://$(find test_robot)/meshes/J4_link.STL; visual mesh filename=file://$(find test_robot)/meshes/J4_link.STL
- link J5_link: geometry collision mesh filename=file://$(find test_robot)/meshes/J5_link.STL; visual mesh filename=file://$(find test_robot)/meshes/J5_link.STL
- link J6_link: geometry collision mesh filename=file://$(find test_robot)/meshes/J6_link.STL; visual mesh filename=file://$(find test_robot)/meshes/J6_link.STL
- link J7_link: geometry collision mesh filename=file://$(find test_robot)/meshes/J7_link.STL; visual mesh filename=file://$(find test_robot)/meshes/J7_link.STL
- link left_after_link: geometry collision mesh filename=file://$(find test_robot)/meshes/left_after_link.STL; visual mesh filename=file://$(find test_robot)/meshes/left_after_link.STL
- link left_befor_link: geometry collision mesh filename=file://$(find test_robot)/meshes/left_befor_link.STL; visual mesh filename=file://$(find test_robot)/meshes/left_befor_link.STL
- link right_after_link: geometry collision mesh filename=file://$(find test_robot)/meshes/right_after_link.STL; visual mesh filename=file://$(find test_robot)/meshes/right_after_link.STL
- link right_before_link: geometry collision mesh filename=file://$(find test_robot)/meshes/right_before_link.STL; visual mesh filename=file://$(find test_robot)/meshes/right_before_link.STL
- link robot_base_link: geometry collision mesh filename=file://$(find test_robot)/meshes/robot_base_link.STL; visual mesh filename=file://$(find test_robot)/meshes/robot_base_link.STL
Joints:
- joint J1_joint: limit lower=-1.1775 upper=1.1775 effort=0 velocity=0 -> lower=-1.1775 upper=1.1775 effort=4 velocity=4
- joint J2_joint: limit lower=-3.14 upper=3.14 effort=0 velocity=0 -> lower=-3.14 upper=3.14 effort=4 velocity=4
- joint J3_joint: limit lower=-3.14 upper=3.14 effort=0 velocity=0 -> lower=-3.14 upper=3.14 effort=4 velocity=4
- joint J5_joint: limit lower=-3.14 upper=3.14 effort=0 velocity=0 -> lower=-3.14 upper=3.14 effort=4 velocity=4
- joint J6_joint: limit lower=-3.14 upper=3.14 effort=0 velocity=0 -> lower=-3.14 upper=3.14 effort=4 velocity=4

Commit message: feature: 加入了控制器，实现了车车的移动

File: core/robot_model/test_robot/urdf/test_robot.urdf (robot description, URDF)
Before this commit: robot test_robot, 13 links, 12 joints
Links:
- link robot_base_link: mass 3.72431445026937 -> 25.0
