Commit message: feature: 导入的兑换站文件，实现了在namespace中启动move_group

File: core/robot_model/exchange_station/urdf/exchange_station.urdf (robot description, URDF)
Before this commit: robot exchange_station, 15 links, 14 joints
Links:
- added link dummy_link
- link L1: geometry collision mesh filename=file://$(find exchange_station)/meshes/L1.STL; visual mesh filename=file://$(find exchange_station)/meshes/L1.STL
- link L2: geometry collision mesh filename=file://$(find exchange_station)/meshes/L2.STL; visual mesh filename=file://$(find exchange_station)/meshes/L2.STL
- link L2_light: geometry collision mesh filename=file://$(find exchange_station)/meshes/L2_light.STL; visual mesh filename=file://$(find exchange_station)/meshes/L2_light.STL
- link L3: geometry collision mesh filename=file://$(find exchange_station)/meshes/L3.STL; visual mesh filename=file://$(find exchange_station)/meshes/L3.STL
- link L3_light: geometry collision mesh filename=file://$(find exchange_station)/meshes/L3_light.STL; visual mesh filename=file://$(find exchange_station)/meshes/L3_light.STL
- link L4: geometry collision mesh filename=file://$(find exchange_station)/meshes/L4.STL; visual mesh filename=file://$(find exchange_station)/meshes/L4.STL
- link L5: geometry collision mesh filename=file://$(find exchange_station)/meshes/L5.STL; visual mesh filename=file://$(find exchange_station)/meshes/L5.STL
- link L6: geometry collision mesh filename=file://$(find exchange_station)/meshes/L6.STL; visual mesh filename=file://$(find exchange_station)/meshes/L6.STL
- link L7: geometry collision mesh filename=file://$(find exchange_station)/meshes/L7.STL; visual mesh filename=file://$(find exchange_station)/meshes/L7.STL
- link L_R: geometry collision mesh filename=file://$(find exchange_station)/meshes/L_R.STL; visual mesh filename=file://$(find exchange_station)/meshes/L_R.STL
- link L_RFID: geometry collision mesh filename=file://$(find exchange_station)/meshes/L_RFID.STL; visual mesh filename=file://$(find exchange_station)/meshes/L_RFID.STL
- link L_base: geometry collision mesh filename=file://$(find exchange_station)/meshes/L_base.STL; visual mesh filename=file://$(find exchange_station)/meshes/L_base.STL
- link L_base_light: geometry collision mesh filename=file://$(find exchange_station)/meshes/L_base_light.STL; visual mesh filename=file://$(find exchange_station)/meshes/L_base_light.STL
- link L_lighit: geometry collision mesh filename=file://$(find exchange_station)/meshes/L_lighit.STL; visual mesh filename=file://$(find exchange_station)/meshes/L_lighit.STL
- link base_link: geometry collision mesh filename=file://$(find exchange_station)/meshes/base_link.STL; visual mesh filename=file://$(find exchange_station)/meshes/base_link.STL
Joints:
- added joint dummy_joint: type fixed, parent dummy_link, child base_link, origin xyz=0 0 0.15 rpy=0 0 0

Commit message: fix: 修复了不能同时tf2树命名冲突的问题，但是有概率启动失败，应该是启动顺序的问题，多启动几次就好了

File: core/robot_model/exchange_station/urdf/exchange_station.urdf (robot description, URDF)
Before this commit: robot exchange_station, 16 links, 15 joints
Links:
- removed link base_link
- removed link dummy_link
- added link exchange_station_base_link, mass 9.4012E-06; collision mesh filename=file://$(find exchange_station)/meshes/base_link.STL; visual mesh filename=file://$(find exchange_station)/meshes/base_link.STL
- added link exchange_station_dummy_link
Joints:
- joint J1: parent base_link -> exchange_station_base_link
- joint J_base: parent base_link -> exchange_station_base_link
- joint dummy_joint: child base_link -> exchange_station_base_link; parent dummy_link -> exchange_station_dummy_link

Commit message: add: 为兑换站添加了一个新的tf2帧，用于处理兑换框位置设定

File: core/robot_model/exchange_station/urdf/exchange_station.urdf (robot description, URDF)
Before this commit: robot exchange_station, 16 links, 15 joints
Links:
- added link exchange_station_root_link
Joints:
- added joint exchange_station_root_joint: type fixed, parent exchange_station_dummy_link, child exchange_station_root_link, origin xyz=1.4 0 0 rpy=0 0 0

Commit message: add: 为兑换站添加了一个新的tf2帧，用于处理兑换框位置设定

File: core/robot_model/exchange_station/urdf/exchange_station.urdf (robot description, URDF)
Before this commit: robot exchange_station, 17 links, 16 joints
Links:
- added link box_center_link
Joints:
- added joint box_center_joint: type fixed, parent L7, child box_center_link, origin xyz=0.2 0.07 0 rpy=-1.5707963267949 0 1.5707963267949
