Commit message: feature: 实现了全部的仿真功能！

File: core/gazebo_sim/test_robot_sim/config/sensor_config.urdf (robot description, URDF)
Before this commit: robot test_robot, 3 links, 3 joints
Links:
- added link image_sensor_link
Joints:
- added joint image_sensor_joint: type fixed, parent dummy, child image_sensor_link, origin xyz=0 0 0.5 rpy=0 0 0

Commit message: fix: 添加了gazebo中的相机参数 comment: 这个gazebo仿真应该是很难做的了，考虑换一换，至少全局仿真是不行的，又卡又不稳定

File: core/gazebo_sim/test_robot_sim/config/sensor_config.urdf (robot description, URDF)
Before this commit: robot test_robot, 4 links, 4 joints
Links:
- added link image_sensor_real_link
Joints:
- added joint image_sensor_real_joint: type fixed, parent image_sensor_link, child image_sensor_real_link, origin xyz=0 0 0 rpy=0 -1.570796327 0
- joint image_sensor_joint: origin xyz=0 0 0.5 rpy=0 0 0 -> xyz=0 0 0.5 rpy=0 1.570796327 0
